File: ecad/UKMARSBOT_LineSensorBasic/UKMARSBOT_LineSensorBasic.kicad_sch (KiCad schematic)
At the start: 32 parts, among them J1 Conn_01x16, Q1 BC337-40, Q2 BPW85C, Q3 BPW85C, Q4 BPW85C, Q5 BPW85C, Q6 BC337-40

Commit message: Merge V2.1 into main and tag as V2.1.0  (#80)
* Fixed an issue with the transistor schematic being wrong for the wall sensor board.

* Updated PDF's

* Reworked chassis board for production

Board reworked based on known issues from prototype builds.

* Updated Mezzanine for PiPico

Updated for v2.0 board set addressing all issues raised on the prototype board.

* Updated basic line follower board

Updated for v2.0 board set addressing all issues raised on the prototype board.

* Add v2 wall sensor board

Wall sensor updated for Issues raised on prototype builds. Better pin markings added to Line sensor, mezz and chassis boards

* V2 boards as sent to fabrication

* Add table mapping Pico pins to devices and functions

* Update wall sensor board connector to socket and transistor base resistor values

* Updated schematics to includes a new RSONLINE field and populated that field with RSOnline part numbers for most passive components

* More RSONLINE part numbers and start of automated kicad exports

* Bug fix for automation

* Bug fix for automation

* kibot tweak

* kibot tweak 2

* kibot tweak 3 - indent error

* kibot config update

* config update 2

* config update 3

* config update 4

* attempt 5

* attempt 6

* attempt 7

* attempt 8

* Attempt 9

* attempt 10

* docs: update ecad/UKMARSBOT_LineSensorBasic/UKMARSBOT_LineSensorBasic.kicad_pro [skip ci]

* attempt 11

* attempt 12

* docs: update KiCad exports [skip ci]

* attempt 13

* docs: update KiCad exports [skip ci]

* removing out of date PCB renders and schematics. These are now automagically maintained in the docs folder

* Motors values where exporting wrong and added battery so it appears on the BOM
Also removed some silly long auto generated discriptions

* docs: update KiCad exports [skip ci]

* Data Change test

* docs: update KiCad exports [skip ci]

* Config Tweak

* docs: update KiCad exports [skip ci]

* Cap rename to maintain consistancy across all boards

* docs: update KiCad exports [skip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
Parts:
- C1, C2: RSONLINE (none) -> 739-6799
- D1, D2, D7: RSONLINE (none) -> 818-7540
- D4, D5, D6: RSONLINE (none) -> "228-6004 or 228-5562 or 713-3974 or 813-4845"
- H3, H4: now left out of the parts list
- J1: Note (none) -> https://uk.rs-online.com/web/p/pcb-sockets/6816820 Need to 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; RSONLINE (none) -> 681-6820
- Q1, Q6: RSONLINE (none) -> 671-1119
- Q2, Q3, Q4, Q5: RSONLINE (none) -> 815-1263
- R10, R11, R12, R14, R7, R8, R9: RSONLINE (none) -> 707-8211
- R15, R2: RSONLINE (none) -> 707-7634
- R16, R4: RSONLINE (none) -> 707-7745
- R17, R3, R5: RSONLINE (none) -> 707-8580
