File: ecad/UKMARSBOT_LineSensorBasic/UKMARSBOT_LineSensorBasic.kicad_pcb (KiCad board)
At the start: 2 copper layers, 40.5 x 81.4 mm, 32 parts, among them J1 Conn_01x16, Q1 BC337-40, Q2 BPW85C, Q3 BPW85C, Q4 BPW85C, Q5 BPW85C, Q6 BC337-40

Commit message: V2.1 Boards ready for fabrication
Parts:
- C1, C2: footprint Capacitor_THT:CP_Radial_D5.0mm_P2.50mm -> Capacitor_THT:CP_Radial_D6.3mm_P2.50mm
- R1: value 50R -> 47R
- moved R14 2.54 mm to (154.9, 77.5)
Routing:
- net 3v3: track 127.2 -> 129.8 mm
- net Vemit: track 114.1 -> 113.1 mm
- net SEN1AIP: track 104.8 -> 105.6 mm
Other:
- board text added: "2025-08-16"
- board text added: "Version 2.1"
- board text removed: "2025-07-07"
- board text removed: "Version 2.0"
